File: 60WKeyboard.kicad_pcb (KiCad board)
At the start: 4 copper layers, 293.8 x 108.2 mm, 248 parts, among them IC1 USBLC6-2SC6, J1 USB4215-03-A_REVA, J2 Conn_02x01_MountingPin, U1 NRF54L15-QFAA-R, U2 TXB0101DRL, U3 PES12-42S-N0024, Y1 ABM11W-32.0000MHZ-7-D1X-T3, Y2 ECS-.327-7-12-TR

Commit message: v0.2 in dev
MCU change because im stupid and now I have to redo rf. Routed columns. Started routing USB port.
Parts:
- moved R5 248.3 mm to (341.0, 90.6), turned to 90 degrees
- moved R4 248.2 mm to (339.5, 90.6), turned to 90 degrees
- moved R6 244.9 mm to (337.9, 90.1)
- moved R7 243.2 mm to (337.9, 91.2)
- moved C24 234.2 mm to (335.2, 90.1), turned to 180 degrees
- moved C25 232.6 mm to (335.2, 91.2), turned to 180 degrees
- moved IC1 228.6 mm to (315.1, 73.8), turned to -90 degrees
- moved R1 90.6 mm to (165.8, 150.6)
- moved R2 87.9 mm to (163.1, 150.6)
- moved D14 12.2 mm to (328.7, 71.5), turned to 0 degrees
Connections:
- net /USP_DP renamed /USB_DP
Routing:
- net /COL_2: track 0.00 -> 101.3 mm, vias 0 -> 5
- net /COL_10: track 0.00 -> 99.2 mm, vias 0 -> 5
- net /COL_11: track 0.00 -> 99.0 mm, vias 0 -> 5
- net /COL_13: track 0.00 -> 98.4 mm, vias 0 -> 5
- net /COL_6: track 0.00 -> 97.7 mm, vias 0 -> 5
- net /COL_0: track 0.00 -> 97.2 mm, vias 0 -> 5
- net /COL_1: track 0.00 -> 94.7 mm, vias 0 -> 4
- net /COL_12: track 0.00 -> 89.8 mm, vias 0 -> 3
- net /COL_8: track 0.00 -> 77.0 mm, vias 0 -> 4
- net /COL_4: track 0.00 -> 76.7 mm, vias 0 -> 4
- net /COL_7: track 0.00 -> 76.6 mm, vias 0 -> 4
- net /COL_9: track 0.00 -> 76.6 mm, vias 0 -> 4
- net /COL_3: track 0.00 -> 76.5 mm, vias 0 -> 4
- net /COL_5: track 0.00 -> 76.5 mm, vias 0 -> 4
- net VBUS: track 0.00 -> 59.7 mm, vias 0 -> 1
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
Commit message: work towards v0.2
Finished updating schematic. Ported to PCB editor. Need to rethink encoder.
Parts:
- removed FB1: 120, Inductor_SMD:L_0402_1005Metric
- removed U3: PES12-42S-N0024, SamacSys_Parts:PES1242SN0024
- added C28: 100nF, Capacitor_SMD:C_0402_1005Metric, B.Cu at (214.1, 189.9)
- added IC2: USBLC6-2SC6, SamacSys_Parts:SOT95P280X145-6N, B.Cu at (222.6, 186.8)
- C1: value 10uF -> 1uF; footprint Capacitor_SMD:C_0603_1608Metric -> Capacitor_SMD:C_0402_1005Metric; moved to F.Cu
- C10: value 8pF -> 1pF; footprint Capacitor_SMD:C_0402_1005Metric -> Capacitor_SMD:C_0201_0603Metric
- C11: value 2.2uF -> 1.2pF; footprint Capacitor_SMD:C_0402_1005Metric -> Capacitor_SMD:C_0201_0603Metric; moved to F.Cu
- C12: value 2.2nF -> 8pF; moved to F.Cu
- C13: value 10nF -> 8pF; moved to F.Cu
- C14: value 2.2uF -> 8pF; moved to F.Cu
- C16, C9: value 8pF -> 100nF
- C19: footprint Capacitor_SMD:C_0603_1608Metric -> Capacitor_SMD:C_0402_1005Metric
- C2: value 100nF -> 47nF; moved to F.Cu
- C23: value 100nF -> 10uF; footprint Capacitor_SMD:C_0402_1005Metric -> Capacitor_SMD:C_0603_1608Metric
- C24: value 10nF -> 100nF; footprint SamacSys_Parts:CAPC1005X55N -> Capacitor_SMD:C_0402_1005Metric
- C25: footprint SamacSys_Parts:CAPC1005X55N -> Capacitor_SMD:C_0402_1005Metric
- C26: value 100nF -> 10nF
- C3: value 100nF -> 1uF; moved to F.Cu
- C4, C5: moved to F.Cu
- C6: value 1.5pF -> 100pF; footprint Capacitor_SMD:C_0201_0603Metric -> Capacitor_SMD:C_0402_1005Metric
- C7: value 2.0pF -> DNP; footprint Capacitor_SMD:C_0201_0603Metric -> Capacitor_SMD:C_0402_1005Metric
- C8: value 0.3pF -> 100nF; footprint Capacitor_SMD:C_0201_0603Metric -> Capacitor_SMD:C_0402_1005Metric; moved to F.Cu
- IC1: value USBLC6-2SC6 -> nRF52840-QFAA-F-R7; footprint SamacSys_Parts:SOT95P280X145-6N -> SamacSys_Parts:QFN40P600X600X95-49N-D
- L1: value 2.7nH -> 15nH; footprint Inductor_SMD:L_0201_0603Metric -> Inductor_SMD:L_0402_1005Metric
- L2: value 3.5nH -> 10uH; footprint Inductor_SMD:L_0201_0603Metric -> Inductor_SMD:L_0603_1608Metric
- L3: value 3.5nH -> 4.7nH; moved to F.Cu
- L4: value 4.7uH -> 2.2nH; footprint Inductor_SMD:L_0603_1608Metric -> Inductor_SMD:L_0201_0603Metric; moved to F.Cu
- S1, S10, S11, S12, S13, S16, S17, S18, S19, S2, S20, S21, S22, S23, S24, S25, S26, S27, S3, S30, S31, S32, S33, S34, S35, S36, S37, S38, S39, S4, S40, S43, S44, S45, S46, S47, S48, S49, S5, S50, S51, S52, S6, S7, S8, S9: footprint ScottoKeebs_Hotswap:Hotswap_MX_Plated_1.00u -> MX_Hotswap:MX-Hotswap-1U; moved to B.Cu
- S14: footprint ScottoKeebs_Hotswap:Hotswap_MX_Plated_2.00u -> MX_Hotswap:MX-Hotswap-2U; moved to B.Cu
- S15, S28: footprint ScottoKeebs_Hotswap:Hotswap_MX_Plated_1.50u -> MX_Hotswap:MX-Hotswap-1.5U; moved to B.Cu
- S29: footprint ScottoKeebs_Hotswap:Hotswap_MX_Plated_1.75u -> MX_Hotswap:MX-Hotswap-1.75U; moved to B.Cu
- S41, S42: footprint ScottoKeebs_Hotswap:Hotswap_MX_Plated_2.25u -> MX_Hotswap:MX-Hotswap-2.25U; moved to B.Cu
- S53: footprint ScottoKeebs_Hotswap:Hotswap_MX_Plated_2.75u -> MX_Hotswap:MX-Hotswap-2.75U; moved to B.Cu
- S54, S55, S56, S58, S59, S60, S61: footprint ScottoKeebs_Hotswap:Hotswap_MX_Plated_1.25u -> MX_Hotswap:MX-Hotswap-1.25U; moved to B.Cu
- S57: footprint ScottoKeebs_Hotswap:Hotswap_MX_Plated_6.25u -> MX_Hotswap:MX-Hotswap-6.25U; moved to B.Cu
- U1: value NRF54L15-QFAA-R -> PES12-42S-N0024; footprint SamacSys_Parts:QFN40P600X600X90-49N -> SamacSys_Parts:PES1242SN0024
- moved U1 141.2 mm to (348.3, 84.3), turned to 90 degrees
- moved L4 114.8 mm to (244.3, 200.8)
- moved IC1 113.7 mm to (236.1, 155.6)
- moved C11 113.0 mm to (244.3, 197.3)
- moved C1 111.4 mm to (235.9, 197.4)
- moved C4 109.6 mm to (238.7, 197.4)
- moved C13 109.3 mm to (241.6, 199.3)
- moved C5 109.0 mm to (238.7, 199.3)
- moved C2 107.2 mm to (235.9, 199.3)
- moved C3 106.5 mm to (235.9, 201.3)
- moved C14 100.3 mm to (241.6, 201.3)
- moved C12 41.2 mm to (241.6, 197.4), turned to 0 degrees
- moved L3 40.3 mm to (244.3, 199.0), turned to 0 degrees
- moved C8 39.1 mm to (238.7, 201.3)
- moved L1 27.5 mm to (249.8, 173.2)
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Connections:
- net Net-(PMIC1-SW2) renamed /SW2
- C1 pad 1: VDD -> Net-(IC1-DEC4)
- C10 pad 1: /XC2 -> /ANT
- C11 pad 1: /DECD -> Net-(C11-Pad1)
- C12 pad 1: /DECA -> /XC1
- C13 pad 1: /DECA -> /XC2
- C14 pad 1: /DECA -> GND
- C14 pad 2: GND -> /XL1
- C15 pad 2: /XL1 -> /XL2
- C16 pad 1: GND -> +3V3
- C16 pad 2: /XL2 -> GND
- C17 pad 1: /VOUT2 -> +3V3
- C2 pad 1: VDD -> Net-(IC1-DEC4)
- C23 pad 1: +3V3 -> VDD
- C24 pad 1: /ENC_TERMINAL-A -> +3V3
- C25 pad 1: /ENC_TERMINAL-B -> /ENC_TERMINAL-A
- C26 pad 1: GND -> /ENC_TERMINAL-B
- C26 pad 2: +3V3 -> GND
- C27 pad 1: +5V -> GND
- C27 pad 2: GND -> +3V3
- C3 pad 1: VDD -> +3V3
- C4 pad 1: VDD -> +3V3
- C5 pad 1: VDD -> /DEC1
- C6 pad 1: Net-(C6-Pad1) -> Net-(IC1-DEC3)
- C7 pad 1: Net-(C7-Pad1) -> Net-(IC1-DEC4)
- C8 pad 1: /RF -> +3V3
- C9 pad 1: /XC1 -> +3V3
- IC1 pad 1: /USB_DP -> /DEC1
- IC1 pad 2: GND -> /XL1
- IC1 pad 3: /USB_DN -> /XL2
- IC1 pad 4: /USB_MCU_DN -> /SDA
- IC1 pad 5: VBUS -> /SCL
- IC1 pad 6: /USB_MCU_DP -> /ROW_0
- L1 pad 1: /ANT -> Net-(IC1-DEC4)
- L1 pad 2: Net-(C6-Pad1) -> Net-(L1-Pad2)
- L2 pad 1: Net-(C6-Pad1) -> Net-(L1-Pad2)
- L2 pad 2: Net-(C7-Pad1) -> Net-(IC1-DCC)
- L3 pad 1: Net-(C7-Pad1) -> /ANT
- L3 pad 2: /RF -> Net-(C11-Pad1)
- L4 pad 1: /DCC -> Net-(C11-Pad1)
- L4 pad 2: /DECD -> /RF
- L5 pad 1: /VOUT2 -> +3V3
- PMIC1 pad 32: /VOUT2 -> +3V3
- R4 pad 2: Net-(U3-CCW) -> Net-(U1-CCW)
- R5 pad 2: Net-(U3-CW) -> Net-(U1-CW)
- R6 pad 2: Net-(U3-CCW) -> Net-(U1-CCW)
- R7 pad 2: Net-(U3-CW) -> Net-(U1-CW)
- TP6 pad 1: /VOUT2 -> +3V3
Routing:
- net Net-(LED14-DOUT): track 0.00 -> 298.0 mm
- net Net-(U3-CW): track 15.0 -> 0.00 mm
- net Net-(U3-CCW): track 8.82 -> 0.00 mm
- net /XC1: track 6.47 -> 0.02 mm
- net /XC2: track 6.10 -> 0.00 mm
- net GND: track 5.85 -> 0.20 mm, vias 1 -> 0
- net /CC1: track 5.45 -> 1.54 mm
- net VBUS: track 59.7 -> 56.0 mm, vias 1 -> 0
- net /DECA: track 2.79 -> 0.00 mm, vias 1 -> 0
- net /USB_DN: track 5.67 -> 3.09 mm, vias 1 -> 0
- net /RF: track 2.40 -> 0.01 mm
- net /USB_DP: track 6.64 -> 4.45 mm, vias 1 -> 0
- net /RESET: track 1.69 -> 0.00 mm
- net /ROW_4: track 1.67 -> 0.00 mm
- net /ROW_3: track 1.65 -> 0.00 mm
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
Commit message: work on v0.2
Moved USB port a bit to facilitate easier routing of the ESD protection. Connected all diodes to keys. Connected most LEDS together.
Parts:
- moved IC2 143.2 mm to (312.2, 75.1), turned to -90 degrees
- moved J1 0.80 mm to (314.4, 64.2)
Routing:
- net Net-(LED28-DOUT): track 0.00 -> 304.7 mm
- net Net-(LED53-DOUT): track 0.00 -> 297.0 mm
- net Net-(LED41-DOUT): track 0.00 -> 292.0 mm
- net Net-(LED52-DOUT): track 0.00 -> 31.1 mm
- net Net-(LED42-DOUT): track 0.00 -> 26.4 mm
- net Net-(LED40-DOUT): track 0.00 -> 26.4 mm
- net Net-(LED29-DOUT): track 0.00 -> 21.6 mm
- net Net-(LED27-DOUT): track 0.00 -> 19.2 mm
- net Net-(LED15-DOUT): track 0.00 -> 19.2 mm
- net Net-(LED51-DOUT): track 0.00 -> 14.5 mm
- net Net-(LED45-DOUT): track 0.00 -> 14.5 mm
- net Net-(LED38-DOUT): track 0.00 -> 14.5 mm
- net Net-(LED35-DOUT): track 0.00 -> 14.5 mm
- net Net-(LED26-DOUT): track 0.00 -> 14.5 mm
- net Net-(LED20-DOUT): track 0.00 -> 14.5 mm
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Other:
- outline, holes or cut-outs redrawn

Commit message: work towards v0.2
QFAA needs replacement with QIAA
Parts:
- C1, C11, C12, C13, C14, C2, C3, C4, C5, C8, L3, L4: moved to B.Cu
- moved C13 45.4 mm to (218.6, 160.2), turned to 180 degrees
- moved L3 41.4 mm to (225.0, 162.3), turned to -90 degrees
- moved L4 41.1 mm to (225.0, 164.5), turned to -90 degrees
- moved C12 39.6 mm to (221.8, 163.1), turned to -90 degrees
- moved C11 39.1 mm to (224.7, 163.4), turned to 180 degrees
- moved C10 18.9 mm to (224.7, 161.3)
- moved IC1 11.0 mm to (225.2, 156.6)
- moved C1 3.94 mm to (235.9, 201.3)
- moved C14 3.94 mm to (241.6, 197.4)
- moved C3 3.94 mm to (235.9, 197.4)
- moved C4 3.94 mm to (238.7, 201.3)
- moved C8 3.94 mm to (238.7, 197.4)
- moved Y1 1.90 mm to (219.7, 162.2)
- moved E1 0.90 mm to (225.0, 167.6)
Routing:
- net /ROW_1: track 0.00 -> 233.4 mm
- net /ROW_0: track 0.00 -> 228.6 mm
- net /ROW_2: track 0.00 -> 216.7 mm
- net /ROW_3: track 0.00 -> 202.4 mm
- net /ROW_4: track 0.00 -> 119.1 mm
- net GND: track 0.20 -> 4.98 mm
- net /ANT: track 0.00 -> 2.41 mm
- net Net-(C11-Pad1): track 0.00 -> 1.51 mm
- net /RF: track 0.01 -> 1.04 mm

Commit message: v0.3
moving along
everything on board
need to wire chip and batt charger ic
switch matrix mostly done
Parts:
- removed C16, C4, C5, C8, C9: 100nF, Capacitor_SMD:C_0402_1005Metric
- removed C25, C26: 10nF, Capacitor_SMD:C_0402_1005Metric
- removed C3: 1uF, Capacitor_SMD:C_0402_1005Metric
- removed C6: 100pF, Capacitor_SMD:C_0402_1005Metric
- removed C7: DNP, Capacitor_SMD:C_0402_1005Metric
- removed IC1: nRF52840-QFAA-F-R7, SamacSys_Parts:QFN40P600X600X95-49N-D
- removed L1: 15nH, Inductor_SMD:L_0402_1005Metric
- removed L2: 10uH, Inductor_SMD:L_0603_1608Metric
- removed R4, R5, R6, R7: 10K, Resistor_SMD:R_0402_1005Metric
- removed TP4: VBUS, TestPoint:TestPoint_Pad_D2.0mm
- removed U1: PES12-42S-N0024, SamacSys_Parts:PES1242SN0024
- added C29: 100pF, Capacitor_SMD:C_0402_1005Metric, B.Cu at (231.8, 180.5)
- added C30: DNP, Capacitor_SMD:C_0402_1005Metric, B.Cu at (234.4, 180.5)
- added C31: 100nF, Capacitor_SMD:C_0402_1005Metric, B.Cu at (222.5, 166.9)
- added C32: 4.7uF, Capacitor_SMD:C_0402_1005Metric, B.Cu at (233.2, 168.6)
- added C33: 4.7uF, Capacitor_SMD:C_0402_1005Metric, B.Cu at (230.8, 166.6)
- added C34: 4.7uF, Capacitor_SMD:C_0402_1005Metric, B.Cu at (237.8, 172.5)
- added C35: 100nF, Capacitor_SMD:C_0402_1005Metric, B.Cu at (238.8, 172.5)
- added C36: 100nF, Capacitor_SMD:C_0402_1005Metric, B.Cu at (239.8, 172.5)
- added C37: 100nF, Capacitor_SMD:C_0402_1005Metric, B.Cu at (241.0, 172.5)
- added U3: nRF52840, Package_DFN_QFN:Nordic_AQFN-73-1EP_7x7mm_P0.5mm, B.Cu at (227.6, 172.2)
- C2: value 47nF -> 1uF
- C27, R8, U2: moved to B.Cu
- TP1, TP2, TP3, TP5, TP6: moved to F.Cu
- moved C22 215.1 mm to (310.2, 91.2), turned to 180 degrees
- moved C24 193.0 mm to (162.6, 176.6)
- moved R8 174.0 mm to (65.4, 103.1), turned to 180 degrees
- moved C28 172.5 mm to (63.7, 105.5), turned to -90 degrees
- moved U2 172.0 mm to (63.0, 103.7)
- moved C27 167.8 mm to (62.3, 105.5), turned to 90 degrees
- moved C19 68.4 mm to (169.8, 173.1), turned to -90 degrees
- moved C18 66.9 mm to (160.3, 172.0), turned to 90 degrees
- moved C17 63.9 mm to (158.0, 176.8), turned to -90 degrees
- moved C21 59.3 mm to (160.7, 175.7), turned to -90 degrees
- moved C20 59.1 mm to (169.5, 170.9), turned to 90 degrees
- moved R3 57.5 mm to (168.5, 168.0)
- moved C23 52.0 mm to (169.5, 175.8), turned to -90 degrees
- moved L5 44.5 mm to (158.0, 173.6), turned to 90 degrees
- moved C14 35.4 mm to (224.3, 166.5)
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Connections:
- C1 pad 1: Net-(IC1-DEC4) -> GND
- C1 pad 2: GND -> /DEC 4 6
- C2 pad 1: Net-(IC1-DEC4) -> GND
- C2 pad 2: GND -> Net-(U3-VDDH)
Routing:
- net +5V: track 0.00 -> 1130.4 mm, vias 0 -> 59
- net GND: track 4.98 -> 170.0 mm, vias 4 -> 70
- net /USB_MCU_DP: track 0.00 -> 153.5 mm, vias 0 -> 2
- net /USB_MCU_DN: track 0.00 -> 153.1 mm
- net VBUS: track 62.0 -> 202.0 mm
- net /COL_0: track 97.2 -> 12.1 mm
- net /ROW_3: track 202.4 -> 238.1 mm, vias 0 -> 2
- net /ROW_2: track 216.7 -> 247.6 mm, vias 0 -> 2
- net /ROW_0: track 228.6 -> 253.3 mm, vias 0 -> 3
- net /ROW_1: track 233.4 -> 257.2 mm, vias 0 -> 2
- net Net-(LED13-DOUT): track 24.0 -> 5.72 mm, vias 0 -> 2
- net /COL_12: track 89.8 -> 106.0 mm, vias 3 -> 4
- net Net-(LED14-DOUT): track 298.0 -> 283.7 mm, vias 0 -> 2
- net Net-(LED41-DOUT): track 292.0 -> 281.5 mm, vias 0 -> 2
- net /XC2: track 0.00 -> 5.92 mm
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- added copper zone on In1.Cu, net GND
- added copper zone on In2.Cu, net GND
Other:
- board size 293.8 x 108.2 mm -> 293.9 x 108.2 mm
