File: 60WKeyboard.kicad_sch (KiCad schematic)
At the start: 196 parts, among them IC1 SN74AHCT1G125DBVR, J1 Conn_01x02, U1 XIAO-nRF52840-SMD, U2 MCP23017_SO, U3 PEC12R-2217F-S0024

Commit message: v0.1-sch
finished schematic
Parts:
- added R5, R6: 10K, symbol Device:R
- added R7, R8: 2k2, symbol Device:R
- IC1: footprint SOT95P280X145-5N -> SamacSys_Parts:SOT95P280X145-5N
- J1: footprint (none) -> Connector_JST:JST_PH_S2B-PH-SM4-TB_1x02-1MP_P2.00mm_Horizontal
- U3: footprint PEC12R2217FS0024 -> (none)
Connections:
- net +3V3: now also R5.1, R6.1, R7.1, R8.1
- net +5V: now also D100.4 (VDD), D101.4 (VDD), D102.4 (VDD), D103.4 (VDD), D104.4 (VDD), D105.4 (VDD), D106.4 (VDD), D107.4 (VDD), D108.4 (VDD), D109.4 (VDD), D110.4 (VDD), D111.4 (VDD), D112.4 (VDD), D113.4 (VDD), D114.4 (VDD), D115.4 (VDD), D116.4 (VDD), D117.4 (VDD), D118.4 (VDD), D119.4 (VDD), D120.4 (VDD), D121.4 (VDD), D122.4 (VDD), D123.4 (VDD), D124.4 (VDD), D62.4 (VDD), D63.4 (VDD), D64.4 (VDD), D65.4 (VDD), D66.4 (VDD), D67.4 (VDD), D68.4 (VDD), D69.4 (VDD), D70.4 (VDD), D71.4 (VDD), D72.4 (VDD), D73.4 (VDD), D74.4 (VDD), D75.4 (VDD), D76.4 (VDD), D77.4 (VDD), D78.4 (VDD), D79.4 (VDD), D80.4 (VDD), D81.4 (VDD), D82.4 (VDD), D83.4 (VDD), D84.4 (VDD), D85.4 (VDD), D86.4 (VDD), D87.4 (VDD), D88.4 (VDD), D89.4 (VDD), D90.4 (VDD), D91.4 (VDD), D92.4 (VDD), D93.4 (VDD), D94.4 (VDD), D95.4 (VDD), D96.4 (VDD), D97.4 (VDD), D98.4 (VDD), D99.4 (VDD)
- net ENC_SW1: now also U1.7 (P1.11_D6_TX)
- net ENC_SW2: now also R6.2
- net ENC_TERMINAL-A: now also U1.9 (P1.13_D8_SCK)
- net ENC_TERMINAL-B: now also U1.10 (P1.14_D9_MISO)
- net GND: now also D100.2 (VSS), D101.2 (VSS), D102.2 (VSS), D103.2 (VSS), D104.2 (VSS), D105.2 (VSS), D106.2 (VSS), D107.2 (VSS), D108.2 (VSS), D109.2 (VSS), D110.2 (VSS), D111.2 (VSS), D112.2 (VSS), D113.2 (VSS), D114.2 (VSS), D115.2 (VSS), D116.2 (VSS), D117.2 (VSS), D118.2 (VSS), D119.2 (VSS), D120.2 (VSS), D121.2 (VSS), D122.2 (VSS), D123.2 (VSS), D124.2 (VSS), D62.2 (VSS), D63.2 (VSS), D64.2 (VSS), D65.2 (VSS), D66.2 (VSS), D67.2 (VSS), D68.2 (VSS), D69.2 (VSS), D70.2 (VSS), D71.2 (VSS), D72.2 (VSS), D73.2 (VSS), D74.2 (VSS), D75.2 (VSS), D76.2 (VSS), D77.2 (VSS), D78.2 (VSS), D79.2 (VSS), D80.2 (VSS), D81.2 (VSS), D82.2 (VSS), D83.2 (VSS), D84.2 (VSS), D85.2 (VSS), D86.2 (VSS), D87.2 (VSS), D88.2 (VSS), D89.2 (VSS), D90.2 (VSS), D91.2 (VSS), D92.2 (VSS), D93.2 (VSS), D94.2 (VSS), D95.2 (VSS), D96.2 (VSS), D97.2 (VSS), D98.2 (VSS), D99.2 (VSS), U1.11 (P1.15_D10_MOSI), U2.15 (A0), U2.16 (A1), U2.17 (A2)
- net RGB_DIN-3v3: now also U1.1 (P0.02_A0_D0)
- net Row 0: now also U2.27 (GPA6)
- net Row 1: now also U2.28 (GPA7)
- net Row 2: now also U1.2 (P0.03_A1_D1)
- net Row 3: now also U1.3 (P0.28_A2_D2)
- net Row 4: now also U1.4 (P0.29_A3_D3)
- net SCL: now also U1.6 (P0.05_A5_D5_SCL), R7.2
- net SDA: now also U1.5 (P0.04_A4_D4_SDA), R8.2
- net at D91.1 (DOUT): now also D92.3 (DIN)
- net at D91.3 (DIN): now also D90.1 (DOUT)
- net at D65.1 (DOUT): now also D66.3 (DIN)
- net at D65.3 (DIN): now also D64.1 (DOUT)
- net at D68.1 (DOUT): now also D69.3 (DIN)
- net at D68.3 (DIN): now also D67.1 (DOUT)
- net at D116.1 (DOUT): now also D117.3 (DIN)
- net at D116.3 (DIN): now also D115.1 (DOUT)
- net at D108.1 (DOUT): now also D109.3 (DIN)
- net at D108.3 (DIN): now also D107.1 (DOUT)
- net at D106.1 (DOUT): now also D107.3 (DIN)
- net at D106.3 (DIN): now also D105.1 (DOUT)
- net at D99.1 (DOUT): now also D100.3 (DIN)
- net at D99.3 (DIN): now also D98.1 (DOUT)
- net at D69.1 (DOUT): now also D70.3 (DIN)
- net at D64.3 (DIN): now also D63.1 (DOUT)
- net at D90.3 (DIN): now also D89.1 (DOUT)
- net at D95.1 (DOUT): now also D96.3 (DIN)
- net at D95.3 (DIN): now also D94.1 (DOUT)
- net at D70.1 (DOUT): now also D71.3 (DIN)
- net at D110.1 (DOUT): now also D111.3 (DIN)
- net at D110.3 (DIN): now also D109.1 (DOUT)
- net at D117.1 (DOUT): now also D118.3 (DIN)
- net at D76.1 (DOUT): now also D77.3 (DIN)
- net at D76.3 (DIN): now also D75.1 (DOUT)
- net at D74.1 (DOUT): now also D75.3 (DIN)
- net at D74.3 (DIN): now also D73.1 (DOUT)
- net at D80.1 (DOUT): now also D81.3 (DIN)
- net at D80.3 (DIN): now also D79.1 (DOUT)
- net at D101.1 (DOUT): now also D102.3 (DIN)
- net at D101.3 (DIN): now also D100.1 (DOUT)
- net at D83.1 (DOUT): now also D84.3 (DIN)
- net at D83.3 (DIN): now also D82.1 (DOUT)
- net at D112.1 (DOUT): now also D113.3 (DIN)
- net at D112.3 (DIN): now also D111.1 (DOUT)
- net at D123.1 (DOUT): now also D124.3 (DIN)
- net at D123.3 (DIN): now also D122.1 (DOUT)
- net at D122.3 (DIN): now also D121.1 (DOUT)
- net at D97.1 (DOUT): now also D98.3 (DIN)
- net at D97.3 (DIN): now also D96.1 (DOUT)
- net at D103.1 (DOUT): now also D104.3 (DIN)
- net at D103.3 (DIN): now also D102.1 (DOUT)
- net at D62.1 (DOUT): now also D63.3 (DIN)
- net at D81.1 (DOUT): now also D82.3 (DIN)
- net at D115.3 (DIN): now also D114.1 (DOUT)
- net at D72.1 (DOUT): now also D73.3 (DIN)
- net at D72.3 (DIN): now also D71.1 (DOUT)
- net at D121.3 (DIN): now also D120.1 (DOUT)
- net at D118.1 (DOUT): now also D119.3 (DIN)
- net at D88.1 (DOUT): now also D89.3 (DIN)
- net at D88.3 (DIN): now also D87.1 (DOUT)
- net at D105.3 (DIN): now also D104.1 (DOUT)
- net at D120.3 (DIN): now also D119.1 (DOUT)
- net at U2.18 (~{RESET}): now also R5.2
- net INTA: now reaches U2.19 (INTB)
- net INTB: now reaches U2.20 (INTA)
- net at D67.3 (DIN): now also D66.1 (DOUT)
- net at D114.3 (DIN): now also D113.1 (DOUT)
- net at D85.1 (DOUT): now also D86.3 (DIN)
- net at D85.3 (DIN): now also D84.1 (DOUT)
- net at D78.1 (DOUT): now also D79.3 (DIN)
- net at D78.3 (DIN): now also D77.1 (DOUT)
- net at D86.1 (DOUT): now also D87.3 (DIN)
- net at D93.1 (DOUT): now also D94.3 (DIN)
- net at D93.3 (DIN): now also D92.1 (DOUT)
- no-connect marks 0 -> 8
Other:
- moved on the sheet: U3

Commit message: work towards v0.2
Complete rework of design from nrf52840 module to nrf54l15 SOC with custom design. Adding new PMIC - npm1300 and supporting components for better fit on board and power savings.
Parts:
- removed C2: 10nF, symbol Device:C
- removed D1, D10, D11, D12, D13, D14, D15, D16, D17, D18, D19, D2, D20, D21, D22, D23, D24, D25, D26, D27, D28, D29, D3, D30, D31, D32, D33, D34, D35, D36, D37, D38, D39, D4, D40, D41, D42, D43, D44, D45, D46, D47, D48, D49, D5, D50, D51, D52, D53, D54, D55, D56, D57, D58, D59, D6, D60, D61, D7, D8, D9: Diode, symbol ScottoKeebs:Placeholder_Diode
- removed D100, D101, D102, D103, D104, D105, D106, D107, D108, D109, D110, D111, D112, D113, D114, D115, D116, D117, D118, D119, D120, D121, D122, D123, D124, D62, D63, D64, D65, D66, D67, D68, D69, D70, D71, D72, D73, D74, D75, D76, D77, D78, D79, D80, D81, D82, D83, D84, D85, D86, D87, D88, D89, D90, D91, D92, D93, D94, D95, D96, D97, D98, D99: SK6812MINI, ScottoKeebs_Components:LED_SK6812MINI, symbol LED:SK6812MINI
- removed IC1: SN74AHCT1G125DBVR, SamacSys_Parts:SOT95P280X145-5N, symbol SamacSys_Parts:SN74AHCT1G125DBVR
- removed R1, R2, R3, R4, R6: 10K, symbol Device:R
- removed S1, S10, S11, S12, S13, S14, S15, S16, S17, S18, S19, S2, S20, S21, S22, S23, S24, S25, S26, S27, S28, S29, S3, S30, S31, S32, S33, S34, S35, S36, S37, S38, S39, S4, S40, S41, S42, S43, S44, S45, S46, S47, S48, S49, S5, S50, S51, S52, S53, S54, S55, S56, S57, S58, S59, S6, S60, S61, S7, S8, S9: Keyswitch, symbol ScottoKeebs:Placeholder_Keyswitch
- removed U1: XIAO-nRF52840-SMD, symbol Seeed_Studio_XIAO_Series:XIAO-nRF52840-SMD
- removed U3: PEC12R-2217F-S0024, symbol SamacSys_Parts:PEC12R-2217F-S0024
- added C10, C11, C12, C13, C3: 100nF, symbol Device:C
- added C4: 10nF, SamacSys_Parts:CAPC1005X55N, symbol Device:C
- added C5, C6, C7, C8: 8pF, symbol Device:C
- added C9: 10uF, symbol Device:C
- added H1, H2, H3, H4, H5, H6: MountingHole_Pad, symbol Mechanical:MountingHole_Pad
- added IC1: USBLC6-2SC6, SOT95P280X145-6N, symbol SamacSys_Parts:USBLC6-2SC6
- added J2: USB4215-03-A_REVA, USB4215-03-A_REVA:GCT_USB4215-03-A_REVA, symbol USB4215-03-A_REVA:USB4215-03-A_REVA
- added PMIC1: NPM1300-QEAA-R7, QFN50P500X500X90-33N, symbol SamacSys_Parts:NPM1300-QEAA-R7
- added R10, R11: 2k2, SamacSys_Parts:RESC1005X40N, symbol Device:R
- added R12, R9: 10K, SamacSys_Parts:RESC1005X40N, symbol Device:R
- added SW1: RotaryEncoder, Rotary_Encoder:RotaryEncoder_Bourns_Horizontal_PEC09-2xxxF-Nxxxx, symbol Device:RotaryEncoder
- added U1: NRF54L15-QFAA-R, NRF54L15-QFAA-R:QFN40P600X600X90-49N, symbol NRF54L15-QFAA-R:NRF54L15-QFAA-R
- added Y1: ABM11W-32.0000MHZ-7-D1X-T3, ABM11W300000MHZ4B1UT3, symbol SamacSys_Parts:ABM11W-32.0000MHZ-7-D1X-T3
- added Y2: ECS-.327-7-12-TR, ECS327712TR, symbol SamacSys_Parts:ECS-.327-7-12-TR
- C1: footprint (none) -> SamacSys_Parts:CAPC1005X55N
- R5: footprint (none) -> SamacSys_Parts:RESC1005X40N
- R7, R8: value 2k2 -> 10K; footprint (none) -> SamacSys_Parts:RESC1005X40N
Connections:
- net +3V3: now also R10.1, R11.1, R12.1, R9.1; no longer R5.1, R7.1
- net ENC_TERMINAL-A: now also R5.1
- net ENC_TERMINAL-B: now also R7.1, C4.1
- net GND: now also C10.2, C11.2, C12.2, C13.2, C3.2, C4.2, C5.2, C6.1, C7.1, C8.2, C9.2, IC1.2 (GND), J2.A1_B12 (GND_A), J2.B1_A12 (GND_B), J2.SH1 (SHIELD), J2.SH2 (SHIELD__1), J2.SH3 (SHIELD__2), J2.SH4 (SHIELD__3), SW1.C, Y1.2 (GND_1), Y1.4 (GND_2)
- net SCL: now also R11.2; no longer R7.2
- net SDA: now also R10.2; no longer R8.2
- net at R5.2: now also R8.2, SW1.A; no longer U2.18 (~{RESET})
- net Column 0: no longer names the net of U2.1 (GPB0)
- net Column 1: no longer names the net of U2.2 (GPB1)
- net Column 10: no longer names the net of U2.23 (GPA2)
- net Column 11: no longer names the net of U2.24 (GPA3)
- net Column 12: no longer names the net of U2.25 (GPA4)
- net Column 13: no longer names the net of U2.26 (GPA5)
- net Column 2: no longer names the net of U2.3 (GPB2)
- net Column 3: no longer names the net of U2.4 (GPB3)
- net Column 4: no longer names the net of U2.5 (GPB4)
- net Column 5: no longer names the net of U2.6 (GPB5)
- net Column 6: no longer names the net of U2.7 (GPB6)
- net Column 7: no longer names the net of U2.8 (GPB7)
- net Column 8: no longer names the net of U2.21 (GPA0)
- net Column 9: no longer names the net of U2.22 (GPA1)
- net Row 0: no longer names the net of U2.27 (GPA6)
- net Row 1: no longer names the net of U2.28 (GPA7)
- new net: R12.2, R7.2, SW1.B
- new net: R9.2, U2.18 (~{RESET})
- new net CC1: J2.B5 (CC2)
- new net CC2: J2.A5 (CC1)
- new net USB_DN: IC1.3 (I/O2_1), J2.A7 (DN1), J2.B7 (DN2)
- new net USB_MCU_DN: IC1.4 (I/O2_2)
- new net USB_MCU_DP: IC1.6 (I/O1_2)
- new net USP_DP: IC1.1 (I/O1_1), J2.A6 (DP1), J2.B6 (DP2)
- new net VBUS: C3.1, IC1.5 (VBUS), J2.A4_B9 (VBUS_A), J2.B4_A9 (VBUS_B)
- new net VDD: C10.1, C11.1, C12.1, C13.1, C9.1, U1.10 (VDD), U1.22 (VDD__1), U1.36 (VDD__2), U1.47 (VDD__3), U1.48 (VDD__4)
- new net XC1: C5.1, U1.34 (XC1), Y1.1 (X1)
- new net XC2: C8.1, U1.35 (XC2), Y1.3 (X2)
- new net XL1: C6.2, U1.1 (P1.00/XL1), Y2.
- new net XL2: C7.2, U1.2 (P1.01/XL2), Y2.2 (OUT/IN)
- no-connect marks 8 -> 2
Other:
- added sheet LEDs (leds.kicad_sch)
- added sheet Switches (switches.kicad_sch)
- note added: "Rotary Encoder"
- note added: "USB Connection"
- note added: "probably not nee3ded"
- moved on the sheet: J1

Commit message: initial v0.2 schematic
Finished initial schematic. nPM1300 and nRF54l15 are wired up.
Parts:
- removed R10, R11: 2k2, SamacSys_Parts:RESC1005X40N, symbol Device:R
- removed R9: 10K, SamacSys_Parts:RESC1005X40N, symbol Device:R
- removed U2: MCP23017_SO, Package_SO:SOIC-28W_7.5x17.9mm_P1.27mm, symbol Interface_Expansion:MCP23017_SO
- added C14, C15, C26: 2.2uF, symbol Device:C
- added C16: 10nF, symbol Device:C
- added C17: 2.2nF, symbol Device:C
- added C18: 1.5pF, symbol Device:C
- added C19: 2.0pF, symbol Device:C
- added C20: 0.3pF, symbol Device:C
- added C21: 100nF, symbol Device:C
- added C22: 1uF, symbol Device:C
- added C23, C24, C25: 10uF, symbol Device:C
- added E1: AMCA31-2R450G-S1F-T3, AMCA31-2R450G-S1F-T3:XDCR_AMCA31-2R450G-S1F-T3, symbol AMCA31-2R450G-S1F-T3:AMCA31-2R450G-S1F-T3
- added FB1: 120, symbol Device:FerriteBead
- added L1: 4.7uH, symbol Device:L
- added L2: 2.7nH, symbol Device:L
- added L3, L4: 3.5nH, symbol Device:L
- added L5: 2.2uH, symbol Device:L
- added R2: 250k, symbol Device:R
- added R3, R6: 10k, symbol Device:R
- added TP1: USB_VBUS, symbol Connector:TestPoint
- PMIC1: value NPM1300-QEAA-R7 -> NPM1300-QEAA-R
Connections:
- net +3V3: now also PMIC1.12 (VDDIO), C21.1, R3.1, R6.1
- net +BATT: now also PMIC1.19 (VBAT), C26.1
- net CC1: now also J2.A5 (CC1), PMIC1.23 (CC1); no longer J2.B5 (CC2)
- net CC2: now also J2.B5 (CC2), PMIC1.24 (CC2); no longer J2.A5 (CC1)
- net COL_0: now also U1.11 (P2.00)
- net COL_1: now also U1.12 (P2.01)
- net COL_10: now also U1.21 (P2.10/TRACEDATA(3))
- net COL_11: now also U1.5 (P1.04/ASO(0)/AIN0)
- net COL_12: now also U1.6 (P1.05/ASI(0)/RADIO(6)/AIN1)
- net COL_13: now also U1.7 (P1.06/ASO(1)/AIN2)
- net COL_2: now also U1.13 (P2.02)
- net COL_3: now also U1.14 (P2.03)
- net COL_4: now also U1.15 (P2.04)
- net COL_5: now also U1.16 (P2.05)
- net COL_6: now also U1.17 (P2.06/TRACECLK)
- net COL_7: now also U1.18 (P2.07/TRACEDATA(0)/SWO)
- net COL_8: now also U1.19 (P2.08/TRACEDATA(1))
- net COL_9: now also U1.20 (P2.09/TRACEDATA(2))
- net ENC_TERMINAL-A: now also U1.8 (P1.07/ASI(1)/AIN3)
- net ENC_TERMINAL-B: now also U1.9 (P1.08/CLK16M/EXTREF)
- net GND: now also H1.1, H2.1, H3.1, H4.1, H5.1, H6.1, PMIC1.17 (VSET1), PMIC1.18 (NTC), PMIC1.2 (PVSS1), PMIC1.28 (LSIN1/VINLDO1), PMIC1.29 (LSOUT1/VOUTLDO1), PMIC1.30 (LSIN2/VINLDO2), PMIC1.31 (LSOUT2/VOUTLDO2), PMIC1.33 (AVSS), PMIC1.6 (PVSS2), U1.32 (VSS_PA), U1.44 (VSS), U1.49 (VSS__1), C14.2, C15.2, C16.2, C17.2, C18.2, C19.2, C20.2, C21.2, C22.2, C23.2, C24.2, C25.2, C26.2, R2.2
- net RGB_DIN_3V3: now also U1.42 (P1.14/RADIO(5)/AIN7)
- net ROW_0: now also U1.23 (P0.00)
- net ROW_1: now also U1.24 (P0.01)
- net ROW_2: now also U1.27 (P0.02)
- net ROW_3: now also U1.28 (P0.03/GRTCPWM)
- net ROW_4: now also U1.29 (P0.04/GRTCLFCLKOUT)
- net SCL: now also PMIC1.14 (SCL), U1.39 (P1.11/ASO(3)/RADIO(2)/AIN4), R3.2
- net SDA: now also PMIC1.13 (SDA), U1.40 (P1.12/ASI(3)/RADIO(3)/AIN5), R6.2
- net VBUS: now also PMIC1.21 (VBUS), C22.1, TP1.1
- net VDD: now also PMIC1.1 (VOUT1), PMIC1.22 (VBUSOUT), PMIC1.4 (PVDD), C23.1, C24.1
- net GPIO3: now reaches PMIC1.10 (GPIO3)
- net GPIO4: now reaches PMIC1.11 (GPIO4)
- net SHPHLD: now reaches PMIC1.15 (SHPHLD)
- net VSET2: now reaches PMIC1.16 (VSET2)
- net VSET2: now also R2.1
- net +5V: now reaches PMIC1.20 (VSYS)
- net VOUT2: now reaches PMIC1.32 (VOUT2)
- net VOUT2: now also C25.1, L5.1
- net at PMIC1.5 (SW2): now also L5.2
- net GPIO0: now reaches PMIC1.7 (GPIO0)
- net GPIO1: now reaches PMIC1.8 (GPIO1)
- net GPIO2: now reaches PMIC1.9 (GPIO2)
- net SWDIO: now reaches U1.25 (SWDIO)
- net SWDCLK: now reaches U1.26 (SWDCLK)
- net RESET: now reaches U1.30 (~{RESET})
- net ANT: now reaches U1.31 (ANT)
- net ANT: now also L2.1
- net DECA: now reaches U1.33 (DECRF)
- net DECA: now also U1.43 (DECA), C15.1, C16.1, C17.1, FB1.2
- net DECD: now reaches U1.45 (DECD)
- net DECD: now also C14.1, FB1.1, L1.2
- net DCC: now reaches U1.46 (DCC)
- net DCC: now also L1.1
- new net: C18.1, L2.2, L3.1
- new net: C19.1, L3.2, L4.1
- new net RF: C20.1, E1.1, L4.2
- no-connect marks 2 -> 11
Other:
- note added: "LED Connection"
- note added: "Mounting Holes"
- note added: "Net Tie"
- note added: "Only at Bottom Layer"
- note added: "Pin49 (VSS_1)"
- note added: "RF Matching Network and Antenna"
- note added: "Switch Matrix Connection"
- note added: "nPM1300"
- note added: "nRF54l15"
- note removed: "probably not nee3ded"
- moved on the sheet: C1, C10, C11, C12, C13, C3, C4, C5, C6, C7, C8, C9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
