File: 60WKeyboard.kicad_sch (KiCad schematic)
At the start: 62 parts, among them IC1 USBLC6-2SC6, IC2 nRF52840-QFAA-F-R7, J1 USB4215-03-A_REVA, J2 Conn_02x01_MountingPin, U1 NRF54L15-QFAA-R, U3 PES12-42S-N0024, Y1 ABM11W-32.0000MHZ-7-D1X-T3, Y2 ECS-.327-7-12-TR

Commit message: work towards v0.2
Finished updating schematic. Ported to PCB editor. Need to rethink encoder.
Parts:
- removed C11, C14: 2.2uF, Capacitor_SMD:C_0402_1005Metric, symbol Device:C
- removed C12: 2.2nF, Capacitor_SMD:C_0402_1005Metric, symbol Device:C
- removed C13: 10nF, Capacitor_SMD:C_0402_1005Metric, symbol Device:C
- removed FB1: 120, Inductor_SMD:L_0402_1005Metric, symbol Device:FerriteBead
- removed U1: NRF54L15-QFAA-R, SamacSys_Parts:QFN40P600X600X90-49N, symbol NRF54L15-QFAA-R:NRF54L15-QFAA-R
- added C16, C9: 100nF, Capacitor_SMD:C_0402_1005Metric, symbol Device:C
- added C23: 10uF, Capacitor_SMD:C_0603_1608Metric, symbol Device:C
- added C6: 100pF, Capacitor_SMD:C_0402_1005Metric, symbol Device:C
- added C7: DNP, Capacitor_SMD:C_0402_1005Metric, symbol Device:C
- C1: value 10uF -> 1uF; footprint Capacitor_SMD:C_0603_1608Metric -> Capacitor_SMD:C_0402_1005Metric
- C10: renamed from C6; value 1.5pF -> 1pF
- C11: renamed from C7; value 2.0pF -> 1.2pF
- C19: footprint Capacitor_SMD:C_0603_1608Metric -> Capacitor_SMD:C_0402_1005Metric
- C2: value 100nF -> 47nF
- C25: renamed from C24; footprint SamacSys_Parts:CAPC1005X55N -> Capacitor_SMD:C_0402_1005Metric
- C26: renamed from C25; footprint SamacSys_Parts:CAPC1005X55N -> Capacitor_SMD:C_0402_1005Metric
- C3: value 100nF -> 1uF
- C8: value 0.3pF -> 100nF; footprint Capacitor_SMD:C_0201_0603Metric -> Capacitor_SMD:C_0402_1005Metric
- IC1: renamed from IC2; footprint QFN40P600X600X95-49N-D -> SamacSys_Parts:QFN40P600X600X95-49N-D
- L1: value 2.7nH -> 15nH; footprint Inductor_SMD:L_0201_0603Metric -> Inductor_SMD:L_0402_1005Metric
- L2: value 3.5nH -> 10uH; footprint Inductor_SMD:L_0201_0603Metric -> Inductor_SMD:L_0603_1608Metric
- L3: value 3.5nH -> 4.7nH
- L4: value 4.7uH -> 2.2nH; footprint Inductor_SMD:L_0603_1608Metric -> Inductor_SMD:L_0201_0603Metric
- renumbered C9 to C12, C10 to C13, C15 to C14, C16 to C15, C23 to C24, IC1 to IC2, U3 to U1
Connections:
- net DECD is gone; now on net RF: L4.2
- net VOUT2 is gone; now on net +3V3: C17.1, L5.1, PMIC1.32 (VOUT2), TP6.1
- net +3V3: now also C3.1, C4.1, C8.1, IC1.12 (VDD_1), IC1.17 (VDD_2), IC1.25 (VDD_3), IC1.37 (VDD_4), IC1.48 (VDD_5), C16.1, C9.1
- net ANT: now also C10.1, IC1.31 (ANT), L3.1; no longer L1.1
- net COL_0: now also IC1.44 (P0.31/AIN7)
- net COL_1: now also IC1.43 (P0.30/AIN6)
- net COL_10: now also IC1.18 (P0.19)
- net COL_11: now also IC1.13 (P0.13)
- net COL_12: now also IC1.14 (P0.14)
- net COL_13: now also IC1.15 (P0.17)
- net COL_2: now also IC1.42 (P0.29/AIN5)
- net COL_3: now also IC1.41 (P0.28/AIN4)
- net COL_4: now also IC1.40 (P0.02/AIN0)
- net COL_5: now also IC1.39 (P0.03/AIN1)
- net COL_6: now also IC1.38 (P1.15)
- net COL_7: now also IC1.21 (P0.22)
- net COL_8: now also IC1.20 (P0.21)
- net COL_9: now also IC1.19 (P0.20)
- net ENC_TERMINAL-A: now also IC1.22 (P0.23)
- net ENC_TERMINAL-B: now also IC1.23 (P0.24)
- net GND: now also IC1.32 (VSS_PA), IC1.45 (VSS_1), IC1.49 (VSS_2), C16.2, C23.2, C6.2, C7.2, C9.2
- net RESET: now also IC1.16 (P0.18/NRESET)
- net RF: no longer C8.1, L3.2
- net RGB_DIN_3V3: now also IC1.24 (P1.00/TRACEDATA0)
- net ROW_0: now also IC1.6 (P0.07/TRACECLK)
- net ROW_1: now also IC1.7 (P0.08)
- net ROW_2: now also IC1.8 (P1.08)
- net ROW_3: now also IC1.9 (P1.09/TRACEDATA3)
- net ROW_4: now also IC1.10 (P0.11/TRACEDATA2)
- net SCL: now also IC1.5 (P0.05/AIN3)
- net SDA: now also IC1.4 (P0.04/AIN2)
- net SWDCLK: now also IC1.27 (SWDCLK)
- net SWDIO: now also IC1.26 (SWDIO)
- net VDD: now also C23.1; no longer C1.1, C2.1, C3.1, C4.1, C5.1
- net XC1: now also C12.1, IC1.35 (XC1), Y1.1 (X1)
- net XC2: now also C13.1, IC1.36 (XC2), Y1.3 (X2)
- net XL1: now also C14.2, IC1.2 (P0.00/XL1), Y2.1
- net XL2: now also C15.2, IC1.3 (P0.01/XL2), Y2.2
- net at L1.2, L2.1: no longer C10.1
- net SW2: now reaches L5.2, PMIC1.5 (SW2)
- net DEC1: now reaches IC1.1 (DEC1)
- net DEC1: now also C5.1
- net at IC1.33 (DEC6): now also C1.1, C2.1, IC1.46 (DEC4), L1.1, C7.1
- net at IC1.34 (DEC3): now also C6.1
- net at IC1.47 (DCC): now also L2.2
- net DCC: no longer names the net of L4.1
- net DCC: now also C11.1, L3.2
- no-connect marks 11 -> 9
Other:
- note added: "Crystals"
- note added: "Ground to PVSS2"
- note added: "check for alternative that fits or drop"
- note added: "nRF52840"
- note removed: "Pin49 (VSS_1)"
- note removed: "nRF54l15"
- moved on the sheet: C10, C11, C12, C13, C14, C15, E1, IC1, Y1, Y2

Commit message: more work towards v0.2
Parts:
- removed L1: 15nH, Inductor_SMD:L_0402_1005Metric, symbol Device:L
- removed L2: 10uH, Inductor_SMD:L_0603_1608Metric, symbol Device:L
- removed TP4: VBUS, TestPoint:TestPoint_Pad_D2.0mm, symbol Connector:TestPoint
- added C29: 100pF, Capacitor_SMD:C_0402_1005Metric, symbol Device:C
- added C30: DNP, Capacitor_SMD:C_0402_1005Metric, symbol Device:C
- added C31, C35, C36, C37: 100nF, Capacitor_SMD:C_0402_1005Metric, symbol Device:C
- added C32, C33, C34: 4.7uF, Capacitor_SMD:C_0402_1005Metric, symbol Device:C
- added U3: nRF52840, Package_DFN_QFN:Nordic_AQFN-73-1EP_7x7mm_P0.5mm, symbol MCU_Nordic:nRF52840
- C2: value 47nF -> 1uF
Connections:
- net ANT: now also U3.H23 (ANT); no longer IC1.31 (ANT)
- net GND: now also C1.1, C2.1, C29.2, C30.2, C31.1, C32.2, C33.2, C34.2, C35.2, C36.2, C37.2, U3.B7 (VSS), U3.EP (VSS), U3.F23 (VSS_PA); no longer C1.2, C2.2, IC1.45 (VSS_1)
- net RESET: now also U3.AC13 (P0.18/~{RESET}); no longer IC1.16 (P0.18/NRESET)
- net SWDCLK: now also U3.AA24 (SWDCLK); no longer IC1.27 (SWDCLK)
- net SWDIO: now also U3.AC24 (SWDIO); no longer IC1.26 (SWDIO)
- net USB_MCU_DN: now also U3.AD4 (D-)
- net USB_MCU_DP: now also U3.AD6 (D+)
- net VBUS: now also C33.1, U3.AD2 (VBUS)
- net XC1: now also U3.B24 (XC1); no longer IC1.35 (XC1)
- net XC2: now also U3.A23 (XC2); no longer IC1.36 (XC2)
- net XL1: now also U3.D2 (XL1/P0.00); no longer IC1.2 (P0.00/XL1)
- net XL2: now also U3.F2 (XL2/P0.01); no longer IC1.3 (P0.01/XL2)
- net at C7.1, IC1.33 (DEC6), IC1.46 (DEC4): no longer C1.1, C2.1
- new net: C2.2, C34.1, C35.1, C36.1, C37.1, U3.A22 (VDD), U3.AD14 (VDD), U3.AD23 (VDD), U3.B1 (VDD), U3.W1 (VDD), U3.Y2 (VDDH)
- new net DEC 1: C31.2, U3.C1 (DEC1)
- new net DEC 3: C29.1, U3.D23 (DEC3)
- new net DEC 4 6: C1.2, C30.1, U3.B5 (DEC4), U3.E24 (DEC6)
- new net DECUSB: C32.1, U3.AC5 (DECUSB)
- no-connect marks 9 -> 13
Other:
- moved on the sheet: C1

Commit message: v0.3
moving along
everything on board
need to wire chip and batt charger ic
switch matrix mostly done
Parts:
- removed C16, C4, C5, C8, C9: 100nF, Capacitor_SMD:C_0402_1005Metric, symbol Device:C
- removed C3: 1uF, Capacitor_SMD:C_0402_1005Metric, symbol Device:C
- removed C6: 100pF, Capacitor_SMD:C_0402_1005Metric, symbol Device:C
- removed C7: DNP, Capacitor_SMD:C_0402_1005Metric, symbol Device:C
- removed IC1: nRF52840-QFAA-F-R7, SamacSys_Parts:QFN40P600X600X95-49N-D, symbol SamacSys_Parts:nRF52840-QFAA-F-R7
- C25, C26, R4, R5, R6, R7, U1: now not fitted
Connections:
- net COL_0: now also U3.AD8 (P0.13)
- net COL_1: now also U3.AC9 (P0.14)
- net COL_10: now also U3.AD20 (P0.24)
- net COL_11: now also U3.AC21 (P0.25)
- net COL_12: now also U3.G1 (P0.26)
- net COL_13: now also U3.H2 (P0.27)
- net COL_2: now also U3.AD10 (P0.15)
- net COL_3: now also U3.AC11 (P0.16)
- net COL_4: now also U3.AD12 (P0.17)
- net COL_5: now also U3.AC15 (P0.19)
- net COL_6: now also U3.AD16 (P0.20)
- net COL_7: now also U3.AC17 (P0.21)
- net COL_8: now also U3.AD18 (P0.22)
- net COL_9: now also U3.AC19 (P0.23)
- net ROW_0: now also U3.M2 (TRACECLK/P0.07)
- net ROW_1: now also U3.N1 (P0.08)
- net ROW_2: now also U3.L24 (NFC1/P0.09)
- net ROW_3: now also U3.J24 (NFC2/P0.10)
- net ROW_4: now also U3.T2 (TRACEDATA2/P0.11)
- net SCL: now also U3.K2 (AIN3/P0.05)
- net SDA: now also U3.J1 (AIN2/P0.04)
- no-connect marks 13 -> 14
Other:
- title: (none) -> 60% Wireless Keyboard
- moved on the sheet: C1, C10, C11, C12, C13, C14, C15, C17, C18, C19, C2, C20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
