File: switches.kicad_sch (KiCad schematic)
At the start: 122 parts

Commit message: created v0.2 pcb
Started work on v0.2 pcb. Placed switches, LEDS, and Diodes. Working on MCU routing
Parts:
- S14: footprint ScottoKeebs_Hotswap:Hotswap_MX_Plated_1.00u -> ScottoKeebs_Hotswap:Hotswap_MX_Plated_2.00u
- S15, S28: footprint ScottoKeebs_Hotswap:Hotswap_MX_Plated_1.00u -> ScottoKeebs_Hotswap:Hotswap_MX_Plated_1.50u
- S29: footprint ScottoKeebs_Hotswap:Hotswap_MX_Plated_1.00u -> ScottoKeebs_Hotswap:Hotswap_MX_Plated_1.75u
- S41, S42: footprint ScottoKeebs_Hotswap:Hotswap_MX_Plated_1.00u -> ScottoKeebs_Hotswap:Hotswap_MX_Plated_2.25u
- S53: footprint ScottoKeebs_Hotswap:Hotswap_MX_Plated_1.00u -> ScottoKeebs_Hotswap:Hotswap_MX_Plated_2.75u
- S54, S55, S56, S58, S59, S60, S61: footprint ScottoKeebs_Hotswap:Hotswap_MX_Plated_1.00u -> ScottoKeebs_Hotswap:Hotswap_MX_Plated_1.25u
- S57: footprint ScottoKeebs_Hotswap:Hotswap_MX_Plated_1.00u -> ScottoKeebs_Hotswap:Hotswap_MX_Plated_6.25u
Changed lines of the file:
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@@
 			)
 		)
-		(property "Footprint" "ScottoKeebs_Hotswap:Hotswap_MX_Plated_1.00u"
+		(property "Footprint" "ScottoKeebs_Hotswap:Hotswap_MX_Plated_6.25u"
 			(at 132.08 142.24 0)
 			(effects
@@
 			)
 		)
-		(property "Footprint" "ScottoKeebs_Hotswap:Hotswap_MX_Plated_1.00u"
+		(property "Footprint" "ScottoKeebs_Hotswap:Hotswap_MX_Plated_1.25u"
 			(at 68.58 142.24 0)
 			(effects
@@
 			)
 		)
-		(property "Footprint" "ScottoKeebs_Hotswap:Hotswap_MX_Plated_1.00u"
+		(property "Footprint" "ScottoKeebs_Hotswap:Hotswap_MX_Plated_1.50u"
 			(at 220.98 66.04 0)
 			(effects
@@
 			)
 		)
-		(property "Footprint" "ScottoKeebs_Hotswap:Hotswap_MX_Plated_1.00u"
+		(property "Footprint" "ScottoKeebs_Hotswap:Hotswap_MX_Plated_1.75u"
 			(at 55.88 91.44 0)
 			(effects
@@
 			)
 		)
-		(property "Footprint" "ScottoKeebs_Hotswap:Hotswap_MX_Plated_1.00u"
+		(property "Footprint" "ScottoKeebs_Hotswap:Hotswap_MX_Plated_2.25u"
 			(at 55.88 116.84 0)
 			(effects
@@
 			)
 		)
-		(property "Footprint" "ScottoKeebs_Hotswap:Hotswap_MX_Plated_1.00u"
+		(property "Footprint" "ScottoKeebs_Hotswap:Hotswap_MX_Plated_1.25u"
 			(at 195.58 142.24 0)
 			(effects
@@
 			)
 		)
-		(property "Footprint" "ScottoKeebs_Hotswap:Hotswap_MX_Plated_1.00u"
+		(property "Footprint" "ScottoKeebs_Hotswap:Hotswap_MX_Plated_2.00u"
 			(at 220.98 40.64 0)
 			(effects
@@
 			)
 		)
-		(property "Footprint" "ScottoKeebs_Hotswap:Hotswap_MX_Plated_1.00u"
+		(property "Footprint" "ScottoKeebs_Hotswap:Hotswap_MX_Plated_1.25u"
 			(at 220.98 142.24 0)
 			(effects
@@
 			)
 		)
-		(property "Footprint" "ScottoKeebs_Hotswap:Hotswap_MX_Plated_1.00u"
+		(property "Footprint" "ScottoKeebs_Hotswap:Hotswap_MX_Plated_1.25u"
 			(at 55.88 142.24 0)
 			(effects
@@
 			)
 		)
-		(property "Footprint" "ScottoKeebs_Hotswap:Hotswap_MX_Plated_1.00u"
+		(property "Footprint" "ScottoKeebs_Hotswap:Hotswap_MX_Plated_1.25u"
 			(at 81.28 142.24 0)
 			(effects
@@
 			)
 		)
-		(property "Footprint" "ScottoKeebs_Hotswap:Hotswap_MX_Plated_1.00u"
+		(property "Footprint" "ScottoKeebs_Hotswap:Hotswap_MX_Plated_2.75u"
 			(at 220.98 116.84 0)
 			(effects
@@
 			)
 		)
-		(property "Footprint" "ScottoKeebs_Hotswap:Hotswap_MX_Plated_1.00u"
+		(property "Footprint" "ScottoKeebs_Hotswap:Hotswap_MX_Plated_2.25u"
 			(at 220.98 91.44 0)
 			(effects
@@
 			)
 		)
-		(property "Footprint" "ScottoKeebs_Hotswap:Hotswap_MX_Plated_1.00u"
+		(property "Footprint" "ScottoKeebs_Hotswap:Hotswap_MX_Plated_1.25u"
 			(at 208.28 142.24 0)
 			(effects
@@
 			)
 		)
-		(property "Footprint" "ScottoKeebs_Hotswap:Hotswap_MX_Plated_1.00u"
+		(property "Footprint" "ScottoKeebs_Hotswap:Hotswap_MX_Plated_1.25u"
 			(at 182.88 142.24 0)
 			(effects
@@
 			)
 		)
-		(property "Footprint" "ScottoKeebs_Hotswap:Hotswap_MX_Plated_1.00u"
+		(property "Footprint" "ScottoKeebs_Hotswap:Hotswap_MX_Plated_1.50u"
 			(at 55.88 66.04 0)
 			(effects

Commit message: work towards v0.2
Finished updating schematic. Ported to PCB editor. Need to rethink encoder.
Parts:
- S1, S10, S11, S12, S13, S16, S17, S18, S19, S2, S20, S21, S22, S23, S24, S25, S26, S27, S3, S30, S31, S32, S33, S34, S35, S36, S37, S38, S39, S4, S40, S43, S44, S45, S46, S47, S48, S49, S5, S50, S51, S52, S6, S7, S8, S9: footprint ScottoKeebs_Hotswap:Hotswap_MX_Plated_1.00u -> MX_Hotswap:MX-Hotswap-1U
- S14: footprint ScottoKeebs_Hotswap:Hotswap_MX_Plated_2.00u -> MX_Hotswap:MX-Hotswap-2U
- S15, S28: footprint ScottoKeebs_Hotswap:Hotswap_MX_Plated_1.50u -> MX_Hotswap:MX-Hotswap-1.5U
- S29: footprint ScottoKeebs_Hotswap:Hotswap_MX_Plated_1.75u -> MX_Hotswap:MX-Hotswap-1.75U
- S41, S42: footprint ScottoKeebs_Hotswap:Hotswap_MX_Plated_2.25u -> MX_Hotswap:MX-Hotswap-2.25U
- S53: footprint ScottoKeebs_Hotswap:Hotswap_MX_Plated_2.75u -> MX_Hotswap:MX-Hotswap-2.75U
- S54, S55, S56, S58, S59, S60, S61: footprint ScottoKeebs_Hotswap:Hotswap_MX_Plated_1.25u -> MX_Hotswap:MX-Hotswap-1.25U
- S57: footprint ScottoKeebs_Hotswap:Hotswap_MX_Plated_6.25u -> MX_Hotswap:MX-Hotswap-6.25U

Commit message: v0.3
moving along
everything on board
need to wire chip and batt charger ic
switch matrix mostly done
Other:
- title: (none) -> 60% Wireless Keyboard
Changed lines of the file:
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@@
 	(generator_version "9.0")
 	(paper "A4")
+	(title_block
+		(title "60% Wireless Keyboard")
+		(date "2025-09-20")
+		(rev "v0.3")
+	)
 	(rectangle
 		(start 46.99 19.05)
