File: switches.kicad_sch (KiCad schematic)
At the start: 122 parts

Commit message: v2 is coming along
Parts:
- renumbered D55 to D10, D3 to D11, D17 to D12, D31 to D13, D43 to D14, D56 to D15, D4 to D16, D18 to D17, D32 to D18, D44 to D19, D1 to D2, D5 to D20, D19 to D21, D33 to D22, D45 to D23, D6 to D24, D20 to D25, D34 to D26, D46 to D27, D7 to D28, D21 to D29, D15 to D3, D35 to D30, D47 to D31, D57 to D32, D8 to D33, D22 to D34, D36 to D35, D48 to D36, D9 to D37, D23 to D38, D37 to D39, D29 to D4, D49 to D40, D10 to D41, D24 to D42, D38 to D43, D50 to D44, D11 to D45, D25 to D46, D39 to D47, D51 to D48, D58 to D49, D42 to D5, D12 to D50, D26 to D51, D40 to D52, D52 to D53, D59 to D54, D13 to D55, D27 to D56, D60 to D57, D14 to D58, D28 to D59, D54 to D6, D41 to D60, D53 to D61, D61 to D62, D2 to D7, D16 to D8, D30 to D9, S3 to S10, S17 to S11, S31 to S12, S43 to S13, S56 to S14, S4 to S15, S18 to S16, S32 to S17, S44 to S18, S5 to S19, S15 to S2, S19 to S20, S33 to S21, S45 to S22, S6 to S23, S20 to S24, S34 to S25, S46 to S26, S7 to S27, S21 to S28, S35 to S29, S29 to S3, S47 to S30, S57 to S31, S8 to S32, S22 to S33, S36 to S34, S48 to S35, S9 to S36, S23 to S37, S37 to S38, S49 to S39, S42 to S4, S10 to S40, S24 to S41, S38 to S42, S50 to S43, S11 to S44, S25 to S45, S39 to S46, S51 to S47, S58 to S48, S12 to S49, S54 to S5, S26 to S50, S40 to S51, S59 to S53, S13 to S54, S27 to S55, S60 to S56, S14 to S57, S28 to S58, S41 to S59, S2 to S6, S53 to S60, S16 to S7, S30 to S8, S55 to S9

Commit message: v2 done for real this time
Parts:
- S31: footprint MX_Hotswap:MX-Hotswap-6.25U -> MX_Hotswap:MX-Hotswap-6.25U-ReversedStabilizers
Changed lines of the file:
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@@
 			)
 		)
-		(property "Footprint" "MX_Hotswap:MX-Hotswap-6.25U"
+		(property "Footprint" "MX_Hotswap:MX-Hotswap-6.25U-ReversedStabilizers"
 			(at 132.08 142.24 0)
 			(hide yes)
